Commit message: update boat parametres

File: vrx_2019/worlds/sandisland.xacro (robot description, xacro)
@@ -46,16 +46,6 @@
     </include>
     <include>
-      <name>post_1</name>
-      <pose>173.558 100.809 0.42 0.046 -0.157 0</pose>
-      <uri>model://post</uri>
-    </include>
-    <include>
-      <name>post_2</name>
-      <pose>177.64 90.86 0.3 0.046 -0.157 0</pose>
-      <uri>model://post</uri>
-    </include>
-    <!-- Antenna for communication with the WAM-V -->
-    <include>
-      <pose>175.69 114.29 1.37 0 0 2.00</pose>
+      <name>antena</name>
+      <pose>169.22 110.06 0.47 0.046 -0.157 0</pose>
       <uri>model://antenna</uri>
     </include>
@@ -66,39 +56,4 @@
       <uri>model://ground_station</uri>
     </include>
-    <include>
-      <name>ground_station_1</name>
-      <pose>179.16 113.73 1.55 0 0 3.54</pose>
-      <uri>model://ground_station</uri>
-    </include>
-    <include>
-      <name>ground_station_2</name>
-      <pose>180.61 110.31 1.55 0 0 3.54</pose>
-      <uri>model://ground_station</uri>
-    </include>
-    <include>
-      <name>ground_station_3</name>
-      <pose>182.05 106.83 1.55 0 0 3.54</pose>
-      <uri>model://ground_station</uri>
-    </include>
-    <include>
-      <name>ground_station_4</name>
-      <pose>183.71 103.14 1.55 0 0 3.54</pose>
-      <uri>model://ground_station</uri>
-    </include>
-    <include>
-      <name>ground_station_5</name>
-      <pose>185.28 99.51 1.55 0 0 3.54</pose>
-      <uri>model://ground_station</uri>
-    </include>
-    <include>
-      <name>ground_station_6</name>
-      <pose>186.80 96.02 1.55 0 0 3.54</pose>
-      <uri>model://ground_station</uri>
-    </include>
-    <include>
-      <name>ground_station_7</name>
-      <pose>188.17 92.45 1.55 0 0 3.54</pose>
-      <uri>model://ground_station</uri>
-    </include>
   </xacro:macro>
 </world>

File: wamv_description/urdf/battery.xacro (robot description, xacro)
@@ -4,5 +4,5 @@
     <link name="${namespace}/${prefix}_battery_link">
       <visual name="${prefix}_battery_visual">
-        <origin xyz="0 -1.03 -.45" rpy="0 0 0"/>
+        <origin xyz="0 -0.5 -.45" rpy="0 0 0"/>
         <geometry>
           <mesh filename="package://vrx_gazebo/models/battery/mesh/battery.dae"/>

File: wamv_description/urdf/thrusters/engine.xacro (robot description, xacro)
@@ -6,19 +6,7 @@
       <visual>
         <geometry>
-          <mesh filename="package://wamv_description/models/engine/mesh/engine.dae"/>
+          <mesh filename="package://wamv_description/models/engine/mesh/engine.dae" scale="0.35 0.35 0.35"/>
         </geometry>
       </visual>
-      <collision name="${prefix}_engine_vertical_axis_collision">
-        <origin xyz="-0.16 0 -0.24" rpy="0 0 0" />
-        <geometry>
-          <box size="0.2 0.15 0.83" />
-        </geometry>
-      </collision>
-      <collision name="${prefix}_engine_rear_end_collision">
-        <origin xyz="-0.34 0 0.12" rpy="0 0 0" />
-        <geometry>
-          <box size="0.12 0.15 0.12" />
-        </geometry>
-      </collision>
       <inertial>
         <mass value="15"/>
@@ -29,5 +17,5 @@
       <visual>
         <geometry>
-          <mesh filename="package://wamv_description/models/propeller/mesh/propeller.dae"/>
+          <mesh filename="package://wamv_description/models/propeller/mesh/propeller.dae" scale="0.35 0.35 0.35"/>
         </geometry>
       </visual>
@@ -35,5 +23,5 @@
         <origin xyz="-0.08 0 0" rpy="0 1.57 0" />
         <geometry>
-          <cylinder length="0.18" radius="0.24" />
+          <cylinder length="0.1" radius="0.08" />
         </geometry>
       </collision>

File: wamv_description/urdf/wamv_base.urdf.xacro (robot description, xacro)
@@ -23,15 +23,11 @@
   <link name="${namespace}/dummy_link">
     <visual>
-      <origin xyz="0 0 0.05" rpy="0 0 3.14159" />
+      <origin xyz="0 0 -0.05" rpy="0 0 3.14159" />
       <geometry>
         <mesh filename="package://wamv_description/models/WAM-V-Base/mesh/balsa.dae" scale="0.1 0.1 0.1"/>
       </geometry>
     </visual>
-    <!-- Left base collisions -->
-    <xacro:main_collisions prefix="left" reflect="1" />
-    <!-- Right side collisions -->
-    <xacro:main_collisions prefix="right" reflect="-1" />
     <collision name="base_base">
-      <origin xyz="0 0 0.05" rpy="0 0 3.14159" />
+      <origin xyz="0 0 -0.05" rpy="0 0 3.14159" />
       <geometry>
         <mesh filename="package://wamv_description/models/WAM-V-Base/mesh/balsa.dae" scale="0.1 0.1 0.1"/>
@@ -39,7 +35,7 @@
     </collision>
     <inertial>
-      <!-- From WAM-V spec sheet -->
-      <mass value="180.0"/>
-      <inertia ixx="120.0" ixy="0.0" ixz="0.0" iyy="393" iyz="0.0" izz="446.0"/>
+      <mass value="20.0"/>
+      <inertia ixx="120.0" ixy="0.0" ixz="0.0" iyy="120" iyz="0.0" izz="446.0"/>
+      <!--inertia ixx="120.0" ixy="0.0" ixz="0.0" iyy="393" iyz="0.0" izz="446.0"/-->
     </inertial>
   </link>

File: wamv_gazebo/urdf/components/wamv_camera.xacro (robot description, xacro)
@@ -1,5 +1,5 @@
 <?xml version="1.0"?>
 <robot xmlns:xacro="http://ros.org/wiki/xacro">
-  <xacro:macro name="wamv_camera" params="name x:=0.5 y:=0 z:=1.5 post_z_from:=1.2965 R:=0 P:=0 Y:=0 post_Y:=0 visualize:=False">
+  <xacro:macro name="wamv_camera" params="name x:=10 y:=10 z:=0.8 post_z_from:=0.1 R:=0 P:=0 Y:=0 post_Y:=0 visualize:=false">
     <!-- Define length variables for link positioning -->
     <xacro:property name="platform_z" value="${post_z_from}"/>
@@ -77,5 +77,5 @@
     <link name="${namespace}/${name}_post_arm_link">
       <visual name="${name}_post_arm_visual">
-        <origin xyz="-0.038 0 -0.003" rpy="${radians(-60)} 0 ${-pi/2}"/>
+        <origin xyz="-0.038 0 -0.003" rpy="${radians(-40)} 0 ${-pi/2}"/>
         <geometry>
           <mesh filename="package://vrx_gazebo/models/sensor_post/mesh/sensor_post_arm.dae"/>
@@ -83,5 +83,5 @@
       </visual>
       <collision name="${name}_post_arm_collision">
-        <origin xyz="0 0 0" rpy="${radians(-60)-pi/20} 0 ${-pi/2}"/>
+        <origin xyz="0 0 0" rpy="${radians(-40)-pi/20} 0 ${-pi/2}"/>
         <geometry>
           <cylinder radius="0.008" length="0.065"/>
@@ -89,5 +89,5 @@
       </collision>
       <inertial>
-        <origin xyz="0 0 0" rpy="${radians(-60)-pi/20} 0 ${-pi/2}"/>
+        <origin xyz="0 0 0" rpy="${radians(-40)-pi/20} 0 ${-pi/2}"/>
         <mass value="0.1"/>
         <inertia

File: wamv_gazebo/urdf/components/wamv_gps.xacro (robot description, xacro)
@@ -1,5 +1,5 @@
 <?xml version="1.0" encoding="UTF-8"?>
 <robot xmlns:xacro="http://ros.org/wiki/xacro">
-  <xacro:macro name="wamv_gps" params="name:=gps x:=0.3 y:=0 z:=1.3
+  <xacro:macro name="wamv_gps" params="name:=gps x:=0.3 y:=0 z:=0.4
 				       R:=0 P:=0 Y:=0 update_rate:=15">
     <link name="${namespace}/${name}_link">

File: wamv_gazebo/urdf/components/wamv_imu.xacro (robot description, xacro)
@@ -1,7 +1,7 @@
 <?xml version="1.0"?>
 <robot xmlns:xacro="http://ros.org/wiki/xacro">
-  <xacro:macro name="wamv_imu" params="name:=imu x:=0.3 y:=0.5 z:=1.3 R:=0 P:=0 Y:=0 update_rate:=15">
+  <xacro:macro name="wamv_imu" params="name:=imu x:=0.0 y:=0.0 z:=0 R:=0 P:=0 Y:=0 update_rate:=15">
     <link name="${namespace}/${name}_link">
-      <visual name="${name}_visual">>
+      <visual name="${name}_visual">
         <geometry>
           <box size="0.05 0.025 0.005" />

File: wamv_gazebo/urdf/thruster_layouts/wamv_gazebo_thruster_config.xacro (robot description, xacro)
@@ -13,6 +13,6 @@
       <mappingType>1</mappingType>
       <maxCmd>1.0</maxCmd>
-      <maxForceFwd>150.0</maxForceFwd>
-      <maxForceRev>-150.0</maxForceRev>
+      <maxForceFwd>100.0</maxForceFwd>
+      <maxForceRev>-100.0</maxForceRev>
       <maxAngle>${pi/2}</maxAngle>
     </thruster>

File: wamv_gazebo/urdf/wamv_gazebo.urdf.xacro (robot description, xacro)
@@ -37,6 +37,6 @@
   <!-- === Batteries === -->
   <xacro:include filename="$(find wamv_description)/urdf/battery.xacro"/>
-  <xacro:battery prefix="left" position="0 1 0.45" orientation="0 0 0"/>
-  <xacro:battery prefix="right" position="0 -1 0.45" orientation="0 0 0"/>
+  <xacro:battery prefix="left" position="0.3 0 0.15" orientation="0 0 1.5708"/>
+  <xacro:battery prefix="right" position="-0.3 0 0.15" orientation="0 0 1.5708"/>
   <!-- === Thrusters === -->
   <!-- Use thruster yaml file if given -->
@@ -100,5 +100,5 @@
     <!-- Add a front camera -->
     <xacro:if value="$(arg camera_enabled)">
-      <xacro:wamv_camera name="front_camera" y="0.3" x="0.75" P="${radians(15)}" />
+      <xacro:wamv_camera name="front_camera" y="0" x="0" P="${radians(15)}" />
     </xacro:if>
     <!-- Add simulated GPS -->
