Commit message: add airport

File: vrx_2019/worlds/example_course.world.xacro (robot description, xacro)
@@ -7,5 +7,20 @@
     <!--Waves-->
     <xacro:include filename="$(find wave_gazebo)/world_models/ocean_waves/model.xacro"/>
-    <xacro:ocean_waves/>
+    <xacro:ocean_waves scale="2.5" gain="0.1"/>
+        <xacro:include filename="$(find vrx_gazebo)/worlds/xacros/usv_wind_plugin.xacro"/>
+     <xacro:usv_wind_gazebo
+	direction="270"
+	mean_vel="0"
+	var_gain="2"
+	var_time="1"
+	seed="42">
+      <wind_objs>
+        <wind_obj>
+          <name>wamv</name>
+          <link_name>wamv/base_link</link_name>
+          <coeff_vector>0.5 0.5 .01</coeff_vector>
+        </wind_obj>
+      </wind_objs>
+    </xacro:usv_wind_gazebo>
     <include>
       <uri>model://robotx_navigation_challenge</uri>
@@ -20,4 +35,8 @@
       <pose>55 -50 0 0 0 -1.3</pose>
     </include>
+    <include>
+      <uri>model://helipuerto</uri>
+      <pose>168 114 0.7 0 0 0.3</pose>
+    </include>
     <!-- The 2016 dock with the three placards -->
     <include>
@@ -30,14 +49,4 @@
       <pose>-2 -18 0.0 0 0 0.2</pose>
     </include>
-    <xacro:include filename="$(find vrx_gazebo)/worlds/xacros/usv_wind_plugin.xacro"/>
-    <xacro:usv_wind_gazebo>
-      <wind_objs>
-        <wind_obj>
-          <name>wamv</name>
-          <link_name>wamv/base_link</link_name>
-          <coeff_vector>.5 .5 .33</coeff_vector>
-        </wind_obj>
-      </wind_objs>
-    </xacro:usv_wind_gazebo>
   </world>
 </sdf>

File: vrx_gazebo/worlds/example_course.world.xacro (robot description, xacro)
@@ -23,4 +23,8 @@
       <uri>model://robotx_light_buoy</uri>
       <pose>-511 218 0.25 0 0 3.14</pose>
+    </include>
+    <include>
+      <uri>model://helipuerto</uri>
+      <pose> 169 116 0.6 0 0 3.14</pose>
     </include>
     <!-- The 2022 dock with the placards -->

File: wamv_description/urdf/wamv_base.urdf.xacro (robot description, xacro)
@@ -40,5 +40,5 @@
       </geometry>
     </collision>
-     <visual>
+     <visual name="visual">
       <origin xyz="-0.8 0 0.6" rpy="0 0 0" />
       <geometry>

File: wamv_gazebo/urdf/wamv_gazebo.urdf.xacro (robot description, xacro)
@@ -100,5 +100,5 @@
     <!-- Add a front camera -->
     <xacro:if value="$(arg camera_enabled)">
-      <xacro:wamv_camera name="front_camera" y="0" x="0" P="${radians(15)}" />
+      <xacro:wamv_camera name="front_camera" y="0" x="0.5" P="${radians(1)}" />
     </xacro:if>
     <!-- Add simulated GPS -->

Commit message: add lidar

File: vrx_2019/worlds/example_course.world.xacro (robot description, xacro)
@@ -19,5 +19,10 @@
           <name>wamv</name>
           <link_name>wamv/base_link</link_name>
-          <coeff_vector>0.5 0.5 .01</coeff_vector>
+          <coeff_vector>0.2 0.2 .01</coeff_vector>
+        </wind_obj>
+                <wind_obj>
+          <name>quadrotor</name>
+          <link_name>base_link</link_name>
+          <coeff_vector>0.05 0.05 .01</coeff_vector>
         </wind_obj>
       </wind_objs>

File: wamv_description/urdf/wamv_base.urdf.xacro (robot description, xacro)
@@ -35,5 +35,5 @@
     </collision>
      <visual>
-      <origin xyz="-0.5 0 0.6" rpy="0 0 0" />
+      <origin xyz="-0.5 0 0.52" rpy="0 0 0" />
       <geometry>
         <mesh filename="package://wamv_description/models/WAM-V-Base/mesh/base.dae" scale="0.01 0.01 0.1"/>
@@ -41,5 +41,5 @@
     </visual>
          <collision name="top_base">
-      <origin xyz="-0.5 0 0.6" rpy="0 0 0" />
+      <origin xyz="-0.5 0 0.52" rpy="0 0 0" />
       <geometry>
         <mesh filename="package://wamv_description/models/WAM-V-Base/mesh/base.dae" scale="0.01 0.01 0.1"/>
@@ -47,5 +47,5 @@
     </collision>
     <visual>
-      <origin xyz="-0.55 0.05 0.6001" rpy="0 0 -1.57" />
+      <origin xyz="-0.55 0.05 0.5201" rpy="0 0 -1.57" />
       <geometry>
         <mesh filename="package://wamv_description/models/WAM-V-Base/mesh/heli.dae" scale="0.009 0.009 0.1"/>
@@ -53,5 +53,5 @@
     </visual>
     <!--visual>
-      <origin xyz="-0.55 0 0.601" rpy="0 0 -1.57" />
+      <origin xyz="-0.55 0 0.5201" rpy="0 0 -1.57" />
       <geometry>
         <mesh filename="package://wamv_description/models/WAM-V-Base/mesh/panel.dae" scale="0.009 0.009 0.1"/>

File: wamv_gazebo/urdf/components/sublidar.xacro (robot description, xacro)
@@ -1,13 +1,13 @@
 <?xml version="1.0" encoding="UTF-8"?>
 <robot xmlns:xacro="http://ros.org/wiki/xacro">
-  <xacro:include filename="$(find wamv_gazebo)/urdf/components/wamv_3d_lidar.xacro"/>
-  <xacro:macro name="lidar"
+  <xacro:include filename="$(find wamv_gazebo)/urdf/components/wamv_sub_lidar.xacro"/>
+  <xacro:macro name="sublidar"
                params = "type:='16_beam'
                          name
-                         x:=0.6 y:=0 z:=0.9
+                         x:=0.6 y:=0 z:=-0.3
                          R:=0 P:=0 Y:=0
                          post_Y:=0 post_z_from:=0">
     <xacro:if value="${type == '16_beam'}">
-      <xacro:wamv_3d_lidar name="${name}"
+      <xacro:wamv_sub_lidar name="${name}"
                            x="${x}" y="${y}" z="${z}"
                            R="${R}" P="${P}" Y="${Y}"
@@ -18,5 +18,5 @@
     </xacro:if>
     <xacro:if value="${type == '32_beam'}">
-      <xacro:wamv_3d_lidar name="${name}"
+      <xacro:wamv_sub_lidar name="${name}"
                            x="${x}" y="${y}" z="${z}"
                            R="${R}" P="${P}" Y="${Y}"
@@ -24,6 +24,6 @@
                            vertical_lasers="32"
                            samples="2187"
-                           min_vertical_angle="-0.186"
-                           max_vertical_angle="0.54"/>
+                           min_vertical_angle="0"
+                           max_vertical_angle="0.1"/>
     </xacro:if>
   </xacro:macro>

File: wamv_gazebo/urdf/components/wamv_camera.xacro (robot description, xacro)
@@ -1,5 +1,5 @@
 <?xml version="1.0"?>
 <robot xmlns:xacro="http://ros.org/wiki/xacro">
-  <xacro:macro name="wamv_camera" params="name x:=10 y:=10 z:=0.8 post_z_from:=0.1 R:=0 P:=0 Y:=0 post_Y:=0 visualize:=false">
+  <xacro:macro name="wamv_camera" params="name x:=10 y:=10 z:=0.6 post_z_from:=0.1 R:=0 P:=0 Y:=0 post_Y:=0 visualize:=false">
     <!-- Define length variables for link positioning -->
     <xacro:property name="platform_z" value="${post_z_from}"/>

File: wamv_gazebo/urdf/components/wamv_pinger.xacro (robot description, xacro)
@@ -1,5 +1,5 @@
 <?xml version="1.0"?>
 <robot xmlns:xacro="http://ros.org/wiki/xacro">
-  <xacro:macro name="wamv_pinger" params="name:='pinger' frameId:='wamv/pinger' position:='0 0 0' orientation:='0 0 0'">
+  <xacro:macro name="wamv_pinger" params="name:='pinger' frameId:='wamv/pinger' position:='0 0 0' orientation:='0 1.5 0'">
     <link name="${namespace}/${name}">
       <visual>

File: wamv_gazebo/urdf/components/wamv_planar_lidar.xacro (robot description, xacro)
@@ -1,7 +1,7 @@
 <?xml version="1.0" encoding="UTF-8"?>
 <robot xmlns:xacro="http://ros.org/wiki/xacro">
-  <xacro:macro name="wamv_multibeam_laser" params="name x:=0.5 y:=0 z:=2 R:=0 P:=0 Y:=0">
+  <xacro:macro name="wamv_multibeam_laser" params="name x:=0.0 y:=0 z:=-0.2 R:=0 P:=1.5 Y:=0">
     <link name="${namespace}/${name}_link">
-      <visual name="${name}_visual">>
+      <visual name="${name}_visual">
         <geometry>
           <cylinder radius="0.025" length="0.1" />
@@ -38,7 +38,12 @@
           </range>
         </ray>
-        <plugin name="multibeam_simulator" filename="libgazebo_ros_gpu_laser.so">
+        <!--plugin name="multibeam_simulator" filename="libgazebo_ros_gpu_laser.so">
           <topicName>${namespace}/${sensor_namespace}lidars/${name}/scan</topicName>
           <frameName>${namespace}/${name}_link</frameName>
+        </plugin-->
+        <plugin name="${name}_plugin" filename="libgazebo_ros_velodyne_gpu_laser.so">
+          <topicName>${namespace}/${sensor_namespace}sublidars/${name}/points</topicName>
+          <frameName>${namespace}/${name}_link</frameName>
+          <min_intensity>0</min_intensity>
         </plugin>
       </sensor>

File: wamv_gazebo/urdf/components/wamv_sub_lidar.xacro (robot description, xacro)
@@ -22,11 +22,11 @@
     noise_stddev: Standard deviation of gaussian noise applied to output pointcloud
   -->
-  <xacro:macro name="wamv_3d_lidar" params="name
+  <xacro:macro name="wamv_sub_lidar" params="name
                                             x:=0.7 y:=0 z:=1.8
                                             R:=0 P:=0 Y:=0
                                             post_Y:=0 post_z_from:=1.2965
                                             update_rate:=10 vertical_lasers:=16 samples:=1875 resolution:=0.1
-                                            min_angle:=${-3*pi/4} max_angle:=${3*pi/4}
-                                            min_vertical_angle:=${-pi/12} max_vertical_angle:=${pi/12}
+                                            min_angle:=${0} max_angle:=${0.1}
+                                            min_vertical_angle:=${-pi/2} max_vertical_angle:=${-pi/2}
                                             max_range:=200 noise_stddev:=0.001">
     <!-- Define length variables for link positioning -->
@@ -137,36 +137,34 @@
     </joint>
     <gazebo reference="${namespace}/${name}_link">
-      <sensor type="gpu_ray" name="${name}_sensor">
-        <update_rate>${update_rate}</update_rate>
+           <sensor name="laser" type="ray">
+        <pose>0 0 0 0 1.57079633 0</pose>
         <ray>
           <scan>
             <horizontal>
-              <samples>${samples/resolution}</samples>
-              <resolution>${resolution}</resolution>
-              <min_angle>${min_angle}</min_angle>
-              <max_angle>${max_angle}</max_angle>
+              <samples>1</samples>
+              <resolution>1</resolution>
+              <min_angle>-0</min_angle>
+              <max_angle>0</max_angle>
             </horizontal>
-            <vertical>
-              <samples>${vertical_lasers}</samples>
-              <resolution>1</resolution>
-              <min_angle>${min_vertical_angle}</min_angle>
-              <max_angle>${max_vertical_angle}</max_angle>
-            </vertical>
           </scan>
           <range>
-            <min>0.1</min>
-            <max>${max_range}</max>
+            <min>0.06</min> <!-- do not change: use min_distance (below) for realistic behavior (smaller values cause issues) -->
+            <max>100</max>   <!-- do not change: use min_distance (below) for realistic behavior (bigger values cause issues) -->
+            <resolution>0.01</resolution>
           </range>
           <noise>
             <type>gaussian</type>
             <mean>0.0</mean>
-            <stddev>${noise_stddev}</stddev>
+            <stddev>0.02</stddev>
           </noise>
         </ray>
-        <plugin name="${name}_plugin" filename="libgazebo_ros_velodyne_gpu_laser.so">
-          <topicName>${namespace}/${sensor_namespace}lidars/${name}/points</topicName>
-          <frameName>${namespace}/${name}_link</frameName>
-          <min_intensity>0</min_intensity>
+          <plugin name="lidar_node" filename="libgazebo_ros_laser.so">
+          <robotNamespace></robotNamespace>
+          <topicName>/laser/scan</topicName>
+          <frameName>/lidar_sensor_link</frameName>
         </plugin>
+         <always_on>1</always_on>
+        <update_rate>1</update_rate>
+        <visualize>true</visualize>
       </sensor>
     </gazebo>

File: wamv_gazebo/urdf/macros.xacro (robot description, xacro)
@@ -12,4 +12,6 @@
   <xacro:include filename="$(find wamv_gazebo)/urdf/components/wamv_3d_lidar.xacro" />
   <xacro:include filename="$(find wamv_gazebo)/urdf/components/lidar.xacro" />
+  <xacro:include filename="$(find wamv_gazebo)/urdf/components/wamv_sub_lidar.xacro" />
+  <xacro:include filename="$(find wamv_gazebo)/urdf/components/sublidar.xacro" />
   <xacro:include filename="$(find wamv_gazebo)/urdf/components/wamv_p3d.xacro" />
   <xacro:include filename="$(find wamv_gazebo)/urdf/components/wamv_pinger.xacro" />

File: wamv_gazebo/urdf/wamv_gazebo.urdf.xacro (robot description, xacro)
@@ -100,5 +100,5 @@
     <!-- Add a front camera -->
     <xacro:if value="$(arg camera_enabled)">
-      <xacro:wamv_camera name="front_camera" y="0" x="0.5" P="${radians(1)}" />
+      <xacro:wamv_camera name="front_camera" y="0" x="0.8" P="${radians(1)}" />
     </xacro:if>
     <!-- Add simulated GPS -->
@@ -112,5 +112,6 @@
     <!-- Add 3D LIDAR -->
     <xacro:if value="$(arg lidar_enabled)">
-      <xacro:lidar name="lidar_wamv" y="-0.3" type="16_beam"/>
+      <xacro:lidar name="lidar_wamv" y="-0.0" type="16_beam"/>
+      <xacro:sublidar name="sublidar_wamv" y="-0.0" type="16_beam"/>
     </xacro:if>
     <!-- Add P3D ground truth -->
@@ -120,5 +121,5 @@
     <!-- Add pinger -->
     <xacro:if value="$(arg pinger_enabled)">
-      <xacro:wamv_pinger name="pinger" position="1.0 0 -1.0" />
+      <xacro:wamv_pinger name="pinger" position="0.0 0 -0.2" />
     </xacro:if>
     <!-- Add ball shooter (default pitch angle: ~-60 deg) -->
@@ -142,4 +143,5 @@
       <!-- Add 3D LIDAR -->
       <xacro:lidar name="lidar_wamv" type="16_beam"/>
+      <xacro:sublidar name="sublidar" type="16_beam"/>
       <!-- Add pinger -->
       <xacro:wamv_pinger name="pinger" position="1.0 0 -1.0" />
