Commit message: add drone site

File: wamv_description/urdf/battery.xacro (robot description, xacro)
@@ -10,5 +10,5 @@
       </visual>
       <collision name="${prefix}_battery_collision">
-        <origin xyz="0 0 .15" rpy="0 0 0"/>
+        <origin xyz="0 0.52 0.1" rpy="0 0 0"/>
         <geometry>
           <box size=".6 .4 .31"/>

File: wamv_description/urdf/wamv_base.urdf.xacro (robot description, xacro)
@@ -27,7 +27,4 @@
         <mesh filename="package://wamv_description/models/WAM-V-Base/mesh/balsa.dae" scale="0.1 0.1 0.1"/>
       </geometry>
-      <material name="balsacolor">
-          <color rgba="0.0 1.0 00 1.0" />
-        </material>
     </visual>
     <collision name="base_base">
@@ -37,4 +34,16 @@
       </geometry>
     </collision>
+    <collision name="top_base">
+      <origin xyz="-0.8 0 0.6" rpy="0 0 0" />
+      <geometry>
+        <box size="1.4 1.4 0.03" />
+      </geometry>
+    </collision>
+     <visual>
+      <origin xyz="-0.8 0 0.6" rpy="0 0 0" />
+      <geometry>
+            <box size="1.4 1.4 0.03" />
+        </geometry>
+    </visual>
     <inertial>
       <mass value="20.0"/>
