Commit message: change of usv's model

File: wamv_description/urdf/wamv_base.urdf.xacro (robot description, xacro)
@@ -6,74 +6,4 @@
   <!-- Macro for creating the main collisions as simple shapes. -->
   <xacro:macro name="main_collisions" params="prefix reflect:=1">
-    <!-- Main float -->
-    <collision name="${prefix}_float">
-      <origin xyz="-0.4 ${1.03*reflect} 0.2" rpy="${0*reflect} 1.57 0" />
-      <geometry>
-        <cylinder length="4" radius="0.2" />
-      </geometry>
-    </collision>
-    <collision name="${prefix}_mid_float">
-      <origin xyz="1.85 ${1.03*reflect} 0.3" rpy="${0*reflect} 1.38 0" />
-      <geometry>
-        <cylinder length="0.5" radius="0.17" />
-      </geometry>
-    </collision>
-    <collision name="${prefix}_front_float">
-      <origin xyz="2.3 ${1.03*reflect} 0.4" rpy="${0*reflect} 1.3 0" />
-      <geometry>
-        <cylinder length="0.45" radius="0.12" />
-      </geometry>
-    </collision>
-    <!-- Front beam -->
-    <collision name="front_${prefix}_beam_lower">
-      <origin xyz="0.9 ${0.85*reflect} 1" rpy="${0.78*reflect} 0 0" />
-      <geometry>
-        <cylinder length="0.5" radius="0.04" />
-      </geometry>
-    </collision>
-    <collision name="front_${prefix}_beam_upper">
-      <origin xyz="0.9 ${0.6*reflect} 1.18" rpy="${1.35*reflect} 0 0" />
-      <geometry>
-        <cylinder length="0.2" radius="0.04" />
-      </geometry>
-    </collision>
-    <!-- Mid beam -->
-    <collision name="mid_${prefix}_beam_lower">
-      <origin xyz="-0.65 ${0.99*reflect} 0.7" rpy="${0.1*reflect} 0.25 0" />
-      <geometry>
-        <cylinder length="0.45" radius="0.03" />
-      </geometry>
-    </collision>
-    <collision name="mid_${prefix}_beam_medium">
-      <origin xyz="-0.57 ${0.87*reflect} 1.05" rpy="${0.75*reflect} 0.25 0" />
-      <geometry>
-        <cylinder length="0.32" radius="0.03" />
-      </geometry>
-    </collision>
-    <collision name="mid_${prefix}_beam_upper">
-      <origin xyz="-0.55 ${0.65*reflect} 1.17" rpy="${1.35*reflect} 0.25 0" />
-      <geometry>
-        <cylinder length="0.3" radius="0.03" />
-      </geometry>
-    </collision>
-    <!-- Rear beam -->
-    <collision name="rear_${prefix}_beam_lower">
-      <origin xyz="-0.74 ${1.03*reflect} 0.7" rpy="${0*reflect} -0.15 0" />
-      <geometry>
-        <cylinder length="0.45" radius="0.03" />
-      </geometry>
-    </collision>
-    <collision name="rear_${prefix}_beam_medium">
-      <origin xyz="-0.79 ${0.91*reflect} 1.05" rpy="${0.75*reflect} -0.15 0" />
-      <geometry>
-        <cylinder length="0.32" radius="0.03" />
-      </geometry>
-    </collision>
-    <collision name="rear_${prefix}_beam_upper">
-      <origin xyz="-0.81 ${0.67*reflect} 1.18" rpy="${1.45*reflect} -0.15 0" />
-      <geometry>
-        <cylinder length="0.3" radius="0.03" />
-      </geometry>
-    </collision>
     <!-- Joint -->
     <collision name="${prefix}_joint">
@@ -93,6 +23,7 @@
   <link name="${namespace}/dummy_link">
     <visual>
+      <origin xyz="0 0 0.05" rpy="0 0 3.14159" />
       <geometry>
-        <mesh filename="package://wamv_description/models/WAM-V-Base/mesh/WAM-V-Base.dae"/>
+        <mesh filename="package://wamv_description/models/WAM-V-Base/mesh/balsa.dae" scale="0.1 0.1 0.1"/>
       </geometry>
     </visual>
@@ -101,9 +32,8 @@
     <!-- Right side collisions -->
     <xacro:main_collisions prefix="right" reflect="-1" />
-     <!-- Top base -->
-    <collision name="top_base">
-      <origin xyz="0 -0 1.25" rpy="0 0 0" />
+    <collision name="base_base">
+      <origin xyz="0 0 0.05" rpy="0 0 3.14159" />
       <geometry>
-        <box size="1.85 1 0.1" />
+        <mesh filename="package://wamv_description/models/WAM-V-Base/mesh/balsa.dae" scale="0.1 0.1 0.1"/>
       </geometry>
     </collision>

File: wamv_gazebo/urdf/thruster_layouts/wamv_aft_thrusters.xacro (robot description, xacro)
@@ -2,6 +2,8 @@
 <robot xmlns:xacro="http://ros.org/wiki/xacro">
   <xacro:include filename="$(find wamv_description)/urdf/thrusters/engine.xacro" />
-  <xacro:engine prefix="left" position="-2.373776 1.027135 0.318237" />
-  <xacro:engine prefix="right" position="-2.373776 -1.027135 0.318237" />
+  <xacro:engine prefix="left" position="0.7 0.7 0.318237" />
+  <xacro:engine prefix="right" position="0.7 -0.7 0.318237" />
+  <xacro:engine prefix="left1" position="-0.7 0.7 0.318237" />
+  <xacro:engine prefix="right1" position="-0.7 -0.7 0.318237" />
   <gazebo>
     <plugin name="wamv_gazebo_thrust" filename="libusv_gazebo_thrust_plugin.so">
@@ -12,4 +14,6 @@
       <xacro:wamv_gazebo_thruster_config name="left" />
       <xacro:wamv_gazebo_thruster_config name="right" />
+      <xacro:wamv_gazebo_thruster_config name="left1" />
+      <xacro:wamv_gazebo_thruster_config name="right1" />
     </plugin>
   </gazebo>

File: wamv_gazebo/urdf/thruster_layouts/wamv_gazebo_thruster_config.xacro (robot description, xacro)
@@ -1,5 +1,5 @@
 <?xml version="1.0"?>
 <plugin xmlns:xacro="http://ros.org/wiki/xacro">
-  <xacro:macro  name="wamv_gazebo_thruster_config" params="name enable_angle:=true">
+  <xacro:macro  name="wamv_gazebo_thruster_config" params="name enable_angle:=false">
     <thruster>
       <!-- Required Parameters -->
@@ -13,6 +13,6 @@
       <mappingType>1</mappingType>
       <maxCmd>1.0</maxCmd>
-      <maxForceFwd>250.0</maxForceFwd>
-      <maxForceRev>-100.0</maxForceRev>
+      <maxForceFwd>150.0</maxForceFwd>
+      <maxForceRev>-150.0</maxForceRev>
       <maxAngle>${pi/2}</maxAngle>
     </thruster>

File: wamv_gazebo/urdf/wamv_gazebo.urdf.xacro (robot description, xacro)
@@ -6,6 +6,6 @@
   <xacro:arg name="thruster_config" default="H" />
   <xacro:arg name="camera_enabled" default="false" />
-  <xacro:arg name="gps_enabled" default="false" />
-  <xacro:arg name="imu_enabled" default="false" />
+  <xacro:arg name="gps_enabled" default="true" />
+  <xacro:arg name="imu_enabled" default="true" />
   <xacro:arg name="lidar_enabled" default="false" />
   <xacro:arg name="ground_truth_enabled" default="false" />

Commit message: update boat world

File: wamv_description/urdf/wamv_base.urdf.xacro (robot description, xacro)
@@ -27,4 +27,7 @@
         <mesh filename="package://wamv_description/models/WAM-V-Base/mesh/balsa.dae" scale="0.1 0.1 0.1"/>
       </geometry>
+      <material name="balsacolor">
+          <color rgba="0.0 1.0 00 1.0" />
+        </material>
     </visual>
     <collision name="base_base">

Commit message: add panel and top base

File: wamv_description/urdf/wamv_base.urdf.xacro (robot description, xacro)
@@ -34,16 +34,28 @@
       </geometry>
     </collision>
-    <collision name="top_base">
-      <origin xyz="-0.8 0 0.6" rpy="0 0 0" />
+     <visual>
+      <origin xyz="-0.5 0 0.6" rpy="0 0 0" />
       <geometry>
-        <box size="1.4 1.4 0.03" />
+        <mesh filename="package://wamv_description/models/WAM-V-Base/mesh/base.dae" scale="0.01 0.01 0.1"/>
+      </geometry>
+    </visual>
+         <collision name="top_base">
+      <origin xyz="-0.5 0 0.6" rpy="0 0 0" />
+      <geometry>
+        <mesh filename="package://wamv_description/models/WAM-V-Base/mesh/base.dae" scale="0.01 0.01 0.1"/>
       </geometry>
     </collision>
-     <visual name="visual">
-      <origin xyz="-0.8 0 0.6" rpy="0 0 0" />
+    <visual>
+      <origin xyz="-0.55 0.05 0.6001" rpy="0 0 -1.57" />
       <geometry>
-            <box size="1.4 1.4 0.03" />
-        </geometry>
+        <mesh filename="package://wamv_description/models/WAM-V-Base/mesh/heli.dae" scale="0.009 0.009 0.1"/>
+      </geometry>
     </visual>
+    <!--visual>
+      <origin xyz="-0.55 0 0.601" rpy="0 0 -1.57" />
+      <geometry>
+        <mesh filename="package://wamv_description/models/WAM-V-Base/mesh/panel.dae" scale="0.009 0.009 0.1"/>
+      </geometry>
+    </visual-->
     <inertial>
       <mass value="20.0"/>

Commit message: change wamv

File: wamv_description/urdf/wamv_base.urdf.xacro (robot description, xacro)
@@ -34,22 +34,22 @@
       </geometry>
     </collision>
-     <visual>
+     <!--visual>
       <origin xyz="-0.5 0 0.52" rpy="0 0 0" />
       <geometry>
         <mesh filename="package://wamv_description/models/WAM-V-Base/mesh/base.dae" scale="0.01 0.01 0.1"/>
       </geometry>
-    </visual>
-         <collision name="top_base">
+    </visual-->
+         <!--collision name="top_base">
       <origin xyz="-0.5 0 0.52" rpy="0 0 0" />
       <geometry>
         <mesh filename="package://wamv_description/models/WAM-V-Base/mesh/base.dae" scale="0.01 0.01 0.1"/>
       </geometry>
-    </collision>
-    <visual>
+    </collision-->
+    <!--visual>
       <origin xyz="-0.55 0.05 0.5201" rpy="0 0 -1.57" />
       <geometry>
         <mesh filename="package://wamv_description/models/WAM-V-Base/mesh/heli.dae" scale="0.009 0.009 0.1"/>
       </geometry>
-    </visual>
+    </visual-->
     <!--visual>
       <origin xyz="-0.55 0 0.5201" rpy="0 0 -1.57" />
